File: hardware/Power.kicad_sch (KiCad schematic)
At the start: 28 parts, among them Q1 DMP6180SK3-13, U2 AP66200

Commit message: Board resize in progress
Parts:
- C1: renamed from Cen1; Function (none) -> Cen1
- C10: renamed from Cout3; Function (none) -> Cout3
- C11: renamed from Cmcu1; Function (none) -> Cmcu1
- C2: renamed from Cvcc1; Function (none) -> Cvcc1
- C3: renamed from Cbst1; Function (none) -> Cbst1
- C4: renamed from Cff1; Function (none) -> Cff1
- C5: renamed from Cin1; Function (none) -> Cin1
- C6: renamed from Cout1; Function (none) -> Cout1
- C7: renamed from Cin2; Function (none) -> Cin2
- C8: renamed from Cout2; Function (none) -> Cout2
- C9: renamed from Cin3; Function (none) -> Cin3
- D1: renamed from Dz1; Function (none) -> Dz1
- D2: renamed from TVS1; Function (none) -> TVS1
- F1: Function (none) -> F1
- FB1: Function (none) -> FB1
- J1: renamed from J_dc1; Function (none) -> J_dc1
- L1: Function (none) -> L1
- Q1: Function (none) -> Q1
- R1: renamed from Ren_top1; Function (none) -> Ren_top1
- R2: renamed from Ren_bot1; Function (none) -> Ren_bot1
- R3: renamed from Rg1; Function (none) -> Rg1
- R4: renamed from Rpg1; Function (none) -> Rpg1
- R5: renamed from Rfb_top1; Function (none) -> Rfb_top1
- R6: renamed from Rfb_bot1; Function (none) -> Rfb_bot1
- TP1: Function (none) -> TP1
- TP2: Function (none) -> TP2
- TP3: Function (none) -> TP3
- U1: renamed from U2; Function (none) -> U2
