File: hardware/Power.kicad_sch (KiCad schematic)
At the start: 28 parts, among them J1 DC Connector, Q1 DMP6180SK3-13, U1 AP66200

Commit message: Board resize in progress
Co-Authored-By: Claude Sonnet 5 <noreply@anthropic.com>
Parts:
- F1: value T3A/63V -> T3A5/63V; footprint Fuse:Fuse_1812_4532Metric -> Fuse:Fuse_1206_3216Metric_Pad1.42x1.75mm_HandSolder; LCSC (none) -> C54934567
Changed lines of the file:
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@@
 			)
 		)
-		(property "Value" "T3A/63V"
+		(property "Value" "T3A5/63V"
 			(at 90.17 59.69 90)
 			(show_name no)
@@
 			)
 		)
-		(property "Footprint" "Fuse:Fuse_1812_4532Metric"
+		(property "Footprint" "Fuse:Fuse_1206_3216Metric_Pad1.42x1.75mm_HandSolder"
 			(at 90.17 65.278 90)
 			(hide yes)
@@
 			(at 90.17 63.5 90)
 			(hide yes)
+			(show_name no)
+			(do_not_autoplace no)
+			(effects
+				(font
+					(size 1.27 1.27)
+				)
+			)
+		)
+		(property "LCSC" "C54934567"
+			(at 90.17 63.5 90)
+			(hide yes)
