File: hardware/Power.kicad_sch (KiCad schematic)
At the start: 28 parts, among them J1 DC Connector, Q1 DMP6180SK3-13, U1 AP66200

Commit message: Board resize in progress
Parts:
- C5: MFR EEEFP1H101AP -> (none); MPN (none) -> EEEFP1H101AP
- L1: LCSC (none) -> C48031458; MPN (none) -> ZD0650-8R2M; Manufacturer (none) -> zoomdo electronics

Commit message: Board resize in progress
Parts:
- U1: footprint Package_DFN_QFN:QFN-16-1EP_4x4mm_P0.65mm_EP2.5x2.5mm -> FilamentDryer:AP66200_U-QFN4040-16_EP2.6x2.6mm_P0.65mm
Changed lines of the file:
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@@
 			)
 		)
-		(property "Footprint" "Package_DFN_QFN:QFN-16-1EP_4x4mm_P0.65mm_EP2.5x2.5mm"
+		(property "Footprint" "FilamentDryer:AP66200_U-QFN4040-16_EP2.6x2.6mm_P0.65mm"
 			(at 106.68 128.27 0)
 			(hide yes)
