File: hardware/Power.kicad_sch (KiCad schematic)
At the start: 28 parts, among them J1 DC Connector, Q1 DMP6180SK3-13, U1 AP66200

Commit message: Add MPN/LCSC/Manufacturer fields to components; layout WIP
Co-Authored-By: Claude Sonnet 5 <noreply@anthropic.com>
Claude-Session: https://claude.ai/code/session_01TtYFysfg3KHuTv6C83JsmH
Parts:
- C1: value (none) -> 100n; now left out of the parts list
- C10, TP1, TP2, TP3: now left out of the parts list
- C11, C6, C8: value 22u 25V X5R -> 22u; Dielectric (none) -> X5R; LCSC (none) -> C45783; MPN (none) -> CL21A226MAQNNNE; Manufacturer (none) -> Samsung; Tolerance (none) -> 20%; Voltage (none) -> 25V
- C2: Dielectric (none) -> X7R; LCSC (none) -> C5199872; MPN (none) -> CL10B105KB8NQNC; Manufacturer (none) -> Samsung; Tolerance (none) -> 10%; Voltage (none) -> 50V
- C3: Dielectric (none) -> X7R; LCSC (none) -> C14663; MPN (none) -> CC0603KRX7R9BB104; Manufacturer (none) -> Yageo; Tolerance (none) -> 10%; Voltage (none) -> 50V
- C4: Dielectric (none) -> C0G; LCSC (none) -> C1671; MPN (none) -> CL10C470JB8NNNC; Manufacturer (none) -> Samsung; Tolerance (none) -> 5%; Voltage (none) -> 50V
- C5: value 100uF/50V -> 100u; Dielectric (none) -> Aluminum Electrolytic; Manufacturer (none) -> Samsung; Tolerance (none) -> 20%; Voltage (none) -> 50V
- C7: value 10µF/63V X7R -> 10u; Dielectric (none) -> X7R; LCSC (none) -> C437568; MPN (none) -> GRM32ER71J106KA12L; Manufacturer (none) -> Murata; Tolerance (none) -> 10%; Voltage (none) -> 63V
- C9: value 100nF / 50V -> 100n; Dielectric (none) -> X7R; LCSC (none) -> C14663; MPN (none) -> CC0603KRX7R9BB104; Manufacturer (none) -> Yageo; Tolerance (none) -> 10%; Voltage (none) -> 50V
- D1: LCSC (none) -> C500789; MPN (none) -> BZX84C15-7-F; Manufacturer (none) -> Diodes Incorporated
- D2: LCSC (none) -> C96335; MPN (none) -> SMBJ28A-TR; Manufacturer (none) -> STMicroelectronics
- F1: LCSC C54934567 -> C54934516; MPN (none) -> JFC1206-1300TS; Manufacturer (none) -> Shenzhen JDT Fuse
- FB1: MPN (none) -> HCB3216KF-601T30; Manufacturer (none) -> TAI-TECH
- J1: LCSC (none) -> C144394; MPN (none) -> B3B-XH-A(LF)(SN); Manufacturer (none) -> JST
- Q1: LCSC (none) -> C93034; MPN (none) -> DMP6180SK3-13; Manufacturer (none) -> Diodes Incorporated
- R1, R3, R5: LCSC (none) -> C25803; MPN (none) -> 0603WAF1003T5E; Manufacturer (none) -> UNI-ROYAL(Uniroyal Elec); Power (none) -> 100mW; TCR (none) -> 100ppm/K; Tolerance (none) -> 1%
- R2: value (none) -> 7k87; now left out of the parts list
- R4: Power (none) -> 100mW; TCR (none) -> 100ppm/K; Tolerance (none) -> 1%; now left out of the parts list
- R6: LCSC (none) -> C25967; MPN (none) -> 0603WAF3162T5E; Manufacturer (none) -> UNI-ROYAL(Uniroyal Elec); Power (none) -> 100mW; TCR (none) -> 100ppm/K; Tolerance (none) -> 1%
- U1: LCSC (none) -> C6741205; MPN (none) -> AP66200FVBW-13; Manufacturer (none) -> Diodes Incorporated

Commit message: Add MPN/LCSC/Manufacturer fields to components; layout WIP
Co-Authored-By: Claude Sonnet 5 <noreply@anthropic.com>
Claude-Session: https://claude.ai/code/session_019K6fhgSgEV4SPy8guMLbu9
Parts:
- C5: Manufacturer Samsung -> Panasonic
- F1: value T3A5/63V -> T3A/63V; LCSC C54934516 -> C354897; MPN JFC1206-1300TS -> 1206T3A63V; Manufacturer Shenzhen JDT Fuse -> Walter Elec
Changed lines of the file:
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@@
 			)
 		)
-		(property "Value" "T3A5/63V"
+		(property "Value" "T3A/63V"
 			(at 90.17 59.69 90)
 			(show_name no)
@@
 			)
 		)
-		(property "LCSC" "C54934516"
+		(property "LCSC" "C354897"
 			(at 90.17 63.5 90)
 			(hide yes)
@@
 			)
 		)
-		(property "MPN" "JFC1206-1300TS"
+		(property "MPN" "1206T3A63V"
 			(at 90.17 63.5 90)
 			(hide yes)
@@
 			)
 		)
-		(property "Manufacturer" "Shenzhen JDT Fuse"
+		(property "Manufacturer" "Walter Elec"
 			(at 90.17 63.5 90)
 			(hide yes)
@@
 			)
 		)
-		(property "Manufacturer" "Samsung"
+		(property "Manufacturer" "Panasonic"
 			(at 144.78 69.85 0)
 			(hide yes)

Commit message: Finalize schematic and PCB revision
Co-Authored-By: Claude Sonnet 5 <noreply@anthropic.com>
Connections:
- no-connect marks 0 -> 1
Changed lines of the file:
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@@
 		(color 0 0 0 0)
+	)
+	(no_connect
+		(at 69.85 66.04)
 	)
 	(wire
