File: hardware/Power.kicad_sch (KiCad schematic)
At the start: 28 parts, among them J1 DC Connector, Q1 DMP6180SK3-13, U1 AP66200

Commit message: Update components and footprints for Mouser sourcing
Parts:
- C1: value 100n -> 1u; Dielectric (none) -> X7R; Function Cen1 -> Cvcc1; LCSC (none) -> C5199872; MPN (none) -> GCM188R71E105KA64J; Manufacturer (none) -> Murata Electronics; Tolerance (none) -> 10%; Voltage (none) -> 25V
- C10: value 470u -> 4u7; footprint Capacitor_SMD:CP_Elec_8x10 -> Capacitor_SMD:C_0603_1608Metric; Dielectric (none) -> X5R; Function Cout3 -> C_vdd1; LCSC (none) -> C19666; MPN (none) -> CL10A475KO8NNNC; Manufacturer (none) -> Samsung Electro-Mechanics; Tolerance (none) -> 10%; Voltage (none) -> 16V
- C11: value 22u -> 100n; footprint Capacitor_SMD:C_0805_2012Metric -> Capacitor_SMD:C_0603_1608Metric; Dielectric X5R -> X7R; Function Cmcu1 -> C_vdd2; LCSC C45783 -> C14663; MPN CL21A226MAQNNNE -> CC0603KRX7R9BB104; Manufacturer Samsung -> YAGEO; Tolerance 20% -> 10%; Voltage 25V -> 50V
- C2: value 1u -> 100n; Function Cvcc1 -> Cbst1; LCSC C5199872 -> C14663; MPN CL10B105KB8NQNC -> CC0603KRX7R9BB104; Manufacturer Samsung -> YAGEO
- C3: value 100n -> 47p; Dielectric X7R -> C0G; Function Cbst1 -> Cff1; LCSC C14663 -> C1671; MPN CC0603KRX7R9BB104 -> CL10C470JC8NNNC; Manufacturer Yageo -> Samsung Electro-Mechanics; Tolerance 10% -> 5%; Voltage 50V -> 100V
- C4: value 47p -> 100u; footprint Capacitor_SMD:C_0603_1608Metric -> SamacSys_Parts:EEE0JA331XP; Dielectric C0G -> Aluminum Electrolytic; Function Cff1 -> Cin1; LCSC C1671 -> C401753; MPN CL10C470JB8NNNC -> EEE-FTH101XAP; Manufacturer Samsung -> Panasonic; Tolerance 5% -> 20%
- C5: value 100u -> 22u; footprint JLCPCB:CAP-SMD_BD8.0-L8.3-W8.3-FD -> Capacitor_SMD:C_0805_2012Metric; Dielectric Aluminum Electrolytic -> X5R; Function Cin1 -> Cout1; LCSC C401753 -> C45783; MPN EEEFP1H101AP -> CC0805MKX5R8BB226; Manufacturer Panasonic -> YAGEO; Voltage 50V -> 25V
- C6: value 22u -> 10u; footprint Capacitor_SMD:C_0805_2012Metric -> Capacitor_SMD:C_1210_3225Metric; Dielectric X5R -> X7R; Function Cout1 -> Cin2; LCSC C45783 -> C437568; MPN CL21A226MAQNNNE -> CL32B106KMVNNWE; Manufacturer Samsung -> Samsung Electro-Mechanics; Tolerance 20% -> 10%; Voltage 25V -> 63V
- C7: value 10u -> 22u; footprint Capacitor_SMD:C_1210_3225Metric -> Capacitor_SMD:C_0805_2012Metric; Dielectric X7R -> X5R; Function Cin2 -> Cout2; LCSC C437568 -> C45783; MPN GRM32ER71J106KA12L -> CC0805MKX5R8BB226; Manufacturer Murata -> YAGEO; Tolerance 10% -> 20%; Voltage 63V -> 25V
- C8: value 22u -> 100n; footprint Capacitor_SMD:C_0805_2012Metric -> Capacitor_SMD:C_0603_1608Metric; Dielectric X5R -> X7R; Function Cout2 -> Cin3; LCSC C45783 -> C14663; MPN CL21A226MAQNNNE -> CC0603KRX7R9BB104; Manufacturer Samsung -> YAGEO; Tolerance 20% -> 10%; Voltage 25V -> 50V
- C9: value 100n -> 22u; footprint Capacitor_SMD:C_0603_1608Metric -> Capacitor_SMD:C_0805_2012Metric; Dielectric X7R -> X5R; Function Cin3 -> Cmcu1; LCSC C14663 -> C45783; MPN CC0603KRX7R9BB104 -> CC0805MKX5R8BB226; Manufacturer Yageo -> YAGEO; Tolerance 10% -> 20%; Voltage 50V -> 25V
- D1: value BZX84C15 -> LED_Small; footprint Package_TO_SOT_SMD:SOT-23 -> LED_SMD:LED_0805_2012Metric; Function Dz1 -> D_led1; LCSC C500789 -> C5569446; MPN BZX84C15-7-F -> HSMG-C170; Manufacturer Diodes Incorporated -> Broadcom
- D2: value SMBJ28A -> PMEG6020ER; footprint Diode_SMD:D_SMB -> Diode_SMD:Nexperia_CFP3_SOD-123W; Function TVS1 -> D_heat1; LCSC C96335 -> C98663; MPN SMBJ28A-TR -> PMEG6020ER-QX; Manufacturer STMicroelectronics -> Nexperia
- F1: value T3A/63V -> DC Connector; footprint Fuse:Fuse_1206_3216Metric_Pad1.42x1.75mm_HandSolder -> Connector_JST:JST_XH_B3B-XH-A_1x03_P2.50mm_Vertical; Function F1 -> J_dc1; LCSC C354897 -> C144394; MPN 1206T3A63V -> B3B-XH-A(LF)(SN); Manufacturer Walter Elec -> JST
- FB1: value HCB3216KF-601T30 -> USB4216-03-A; footprint Inductor_SMD:L_1206_3216Metric -> USB421603A; Function FB1 -> (none); LCSC C357023 -> (none); MPN HCB3216KF-601T30 -> USB4216-03-A; Manufacturer TAI-TECH -> GCT; Mouser Part Number (none) -> 640-USB4216-03-A
- J1: value DC Connector -> Sensor; footprint Connector_JST:JST_XH_B3B-XH-A_1x03_P2.50mm_Vertical -> FilamentDryer:JST_PH_B4B-PH-SM4-TB_1x04-1MP_P2.00mm_Vertical; Function J_dc1 -> J_sens1; LCSC C144394 -> C160354; MPN B3B-XH-A(LF)(SN) -> B4B-PH-SM4-TB(LF)(SN)
- L1: value 8u2 -> MMBT3904; footprint JLCPCB:IND-SMD_L7.0-W6.6_ZD0650-100M -> Package_TO_SOT_SMD:SOT-23; Function L1 -> Q_rst1; LCSC C48031458 -> C94514; MPN ZD0650-8R2M -> MMBT3904-7-F; Manufacturer zoomdo electronics -> Diodes Incorporated
- Q1: value DMP6180SK3-13 -> IRLR3636TRPBF; Function Q1 -> Q_heat1; LCSC C93034 -> C67279; MPN DMP6180SK3-13 -> IRLR3636TRPBF; Manufacturer Diodes Incorporated -> Infineon
- R1: value 100k -> 31k6; Function Ren_top1 -> Rfb_bot1; LCSC C25803 -> C25967; MPN 0603WAF1003T5E -> RC0603FR-1331K6L; Manufacturer UNI-ROYAL(Uniroyal Elec) -> YAGEO
- R2: value 7k87 -> 22k1; Function Ren_bot1 -> R_vbus_top1; LCSC (none) -> C25961; MPN (none) -> RC0603FR-1322K1L; Manufacturer (none) -> YAGEO; Power (none) -> 100mW; Tolerance (none) -> 1%
- R3: value 100k -> 47k5; Function Rg1 -> R_vbus_bot1; LCSC C25803 -> C23061; MPN 0603WAF1003T5E -> RC0603FR-0747K5L; Manufacturer UNI-ROYAL(Uniroyal Elec) -> YAGEO
- R4: value 100k -> 1k; Function Rpg1 -> R_rst1; LCSC (none) -> C21190; MPN (none) -> RC0603FR-071KL; Manufacturer (none) -> YAGEO
- R5: value 100k -> 5k1; Function Rfb_top1 -> R_cc2; LCSC C25803 -> C23186; MPN 0603WAF1003T5E -> RC0603FR-075K1L; Manufacturer UNI-ROYAL(Uniroyal Elec) -> YAGEO
- R6: value 31k6 -> 5k1; Function Rfb_bot1 -> R_cc1; LCSC C25967 -> C23186; MPN 0603WAF3162T5E -> RC0603FR-075K1L; Manufacturer UNI-ROYAL(Uniroyal Elec) -> YAGEO

Commit message: Repair symbol fields after CSV import
Parts:
- C1: value 1u -> 100n; Dielectric X7R -> (none); Function Cvcc1 -> Cen1; LCSC C5199872 -> (none); MPN GCM188R71E105KA64J -> (none); Manufacturer Murata Electronics -> (none); Tolerance 10% -> (none); Voltage 25V -> (none)
- C10: value 4u7 -> 470u; footprint Capacitor_SMD:C_0603_1608Metric -> Capacitor_SMD:CP_Elec_8x10; Dielectric X5R -> (none); Function C_vdd1 -> Cout3; LCSC C19666 -> (none); MPN CL10A475KO8NNNC -> (none); Manufacturer Samsung Electro-Mechanics -> (none); Tolerance 10% -> (none); Voltage 16V -> (none)
- C11: value 100n -> 22u; footprint Capacitor_SMD:C_0603_1608Metric -> Capacitor_SMD:C_0805_2012Metric; Dielectric X7R -> X5R; Function C_vdd2 -> Cmcu1; LCSC C14663 -> (none); MPN CC0603KRX7R9BB104 -> CC0805MKX5R8BB226; Tolerance 10% -> 20%; Voltage 50V -> 25V
- C2: value 100n -> 1u; Function Cbst1 -> Cvcc1; LCSC C14663 -> (none); MPN CC0603KRX7R9BB104 -> GCM188R71E105KA64J; Manufacturer YAGEO -> Murata Electronics; Voltage 50V -> 25V
- C3: value 47p -> 100n; Dielectric C0G -> X7R; Function Cff1 -> Cbst1; LCSC C1671 -> C14663; MPN CL10C470JC8NNNC -> CC0603KRX7R9BB104; Manufacturer Samsung Electro-Mechanics -> YAGEO; Tolerance 5% -> 10%; Voltage 100V -> 50V
- C4: value 100u -> 47p; footprint SamacSys_Parts:EEE0JA331XP -> Capacitor_SMD:C_0603_1608Metric; Dielectric Aluminum Electrolytic -> C0G; Function Cin1 -> Cff1; LCSC C401753 -> (none); MPN EEE-FTH101XAP -> CL10C470JC8NNNC; Manufacturer Panasonic -> Samsung Electro-Mechanics; Tolerance 20% -> 5%; Voltage 50V -> 100V
- C5: value 22u -> 100u; footprint Capacitor_SMD:C_0805_2012Metric -> SamacSys_Parts:EEE0JA331XP; Dielectric X5R -> Aluminum Electrolytic; Function Cout1 -> Cin1; LCSC C45783 -> (none); MPN CC0805MKX5R8BB226 -> EEE-FTH101XAP; Manufacturer YAGEO -> Panasonic; Voltage 25V -> 50V
- C6: value 10u -> 22u; footprint Capacitor_SMD:C_1210_3225Metric -> Capacitor_SMD:C_0805_2012Metric; Dielectric X7R -> X5R; Function Cin2 -> Cout1; LCSC C437568 -> (none); MPN CL32B106KMVNNWE -> CC0805MKX5R8BB226; Manufacturer Samsung Electro-Mechanics -> YAGEO; Tolerance 10% -> 20%; Voltage 63V -> 25V
- C7: value 22u -> 10u; footprint Capacitor_SMD:C_0805_2012Metric -> Capacitor_SMD:C_1210_3225Metric; Dielectric X5R -> X7R; Function Cout2 -> Cin2; LCSC C45783 -> (none); MPN CC0805MKX5R8BB226 -> CL32B106KMVNNWE; Manufacturer YAGEO -> Samsung Electro-Mechanics; Tolerance 20% -> 10%; Voltage 25V -> 63V
- C8: value 100n -> 22u; footprint Capacitor_SMD:C_0603_1608Metric -> Capacitor_SMD:C_0805_2012Metric; Dielectric X7R -> X5R; Function Cin3 -> Cout2; LCSC C14663 -> (none); MPN CC0603KRX7R9BB104 -> CC0805MKX5R8BB226; Tolerance 10% -> 20%; Voltage 50V -> 25V
- C9: value 22u -> 100n; footprint Capacitor_SMD:C_0805_2012Metric -> Capacitor_SMD:C_0603_1608Metric; Dielectric X5R -> X7R; Function Cmcu1 -> Cin3; LCSC C45783 -> C14663; MPN CC0805MKX5R8BB226 -> CC0603KRX7R9BB104; Tolerance 20% -> 10%; Voltage 25V -> 50V
- D1: value LED_Small -> BZX84C15; footprint LED_SMD:LED_0805_2012Metric -> Package_TO_SOT_SMD:SOT-23; Function D_led1 -> Dz1; LCSC C5569446 -> C500789; MPN HSMG-C170 -> BZX84C15-7-F; Manufacturer Broadcom -> Diodes Incorporated
- D2: value PMEG6020ER -> SMBJ28A; footprint Diode_SMD:Nexperia_CFP3_SOD-123W -> Diode_SMD:D_SMB; Function D_heat1 -> TVS1; LCSC C98663 -> (none); MPN PMEG6020ER-QX -> SMBJ28A; Manufacturer Nexperia -> Littelfuse
- F1: value DC Connector -> T3A/63V; footprint Connector_JST:JST_XH_B3B-XH-A_1x03_P2.50mm_Vertical -> Fuse:Fuse_1206_3216Metric_Pad1.42x1.75mm_HandSolder; Function J_dc1 -> F1; LCSC C144394 -> (none); MPN B3B-XH-A(LF)(SN) -> SF-1206S300W-2; Manufacturer JST -> Bourns
- FB1: value USB4216-03-A -> BLM31KN601SH1L; footprint USB421603A -> Inductor_SMD:L_1206_3216Metric; Function (none) -> FB1; MPN USB4216-03-A -> BLM31KN601SH1L; Manufacturer GCT -> Murata Electronics; Mouser Part Number 640-USB4216-03-A -> (none)
- J1: value Sensor -> DC Connector; footprint FilamentDryer:JST_PH_B4B-PH-SM4-TB_1x04-1MP_P2.00mm_Vertical -> Connector_JST:JST_XH_B3B-XH-A_1x03_P2.50mm_Vertical; Function J_sens1 -> J_dc1; LCSC C160354 -> C144394; MPN B4B-PH-SM4-TB(LF)(SN) -> B3B-XH-A(LF)(SN)
- L1: value MMBT3904 -> 8u2; footprint Package_TO_SOT_SMD:SOT-23 -> FilamentDryer:XAL4040-822MEC_HandSolder; Function Q_rst1 -> L1; LCSC C94514 -> (none); MPN MMBT3904-7-F -> XAL4040-822MEC; Manufacturer Diodes Incorporated -> Coilcraft
- Q1: value IRLR3636TRPBF -> DMP6180SK3-13; Function Q_heat1 -> Q1; LCSC C67279 -> C93034; MPN IRLR3636TRPBF -> DMP6180SK3-13; Manufacturer Infineon -> Diodes Incorporated
- R1: value 31k6 -> 100k; Function Rfb_bot1 -> Ren_top1; LCSC C25967 -> (none); MPN RC0603FR-1331K6L -> RC0603FR-07100KL
- R2: value 22k1 -> 7k87; Function R_vbus_top1 -> Ren_bot1; LCSC C25961 -> (none); MPN RC0603FR-1322K1L -> (none); Manufacturer YAGEO -> (none); Power 100mW -> (none); Tolerance 1% -> (none)
- R3: value 47k5 -> 100k; Function R_vbus_bot1 -> Rg1; LCSC C23061 -> (none); MPN RC0603FR-0747K5L -> RC0603FR-07100KL
- R4: value 1k -> 100k; Function R_rst1 -> Rpg1; LCSC C21190 -> (none); MPN RC0603FR-071KL -> (none); Manufacturer YAGEO -> (none)
- R5: value 5k1 -> 100k; Function R_cc2 -> Rfb_top1; LCSC C23186 -> (none); MPN RC0603FR-075K1L -> RC0603FR-07100KL
- R6: value 5k1 -> 31k6; Function R_cc1 -> Rfb_bot1; LCSC C23186 -> (none); MPN RC0603FR-075K1L -> RC0603FR-1331K6L
- U1: value AP66200 -> AP66200QFVBW-13; LCSC C6741205 -> (none); MPN AP66200FVBW-13 -> AP66200QFVBW-13

Commit message: Remomved LCSC field
Parts:
- C3, C9: LCSC C14663 -> (none)
- D1: LCSC C500789 -> (none)
- J1: LCSC C144394 -> (none)
- Q1: LCSC C93034 -> (none)
