File: hardware/Filament_Dryer_Monitor.kicad_pcb (KiCad board)
At the start: 4 copper layers, 98 x 58 mm, 91 parts, among them J1 DC Connector, J2 USB_C_Receptacle_USB2.0_16P, J3 Sensor, J4 Display, J5 Heater Connector, J6 Fan Connector, J7 NTC Connector, Q1 DMP6180SK3-13, Q2 MMBT3904, Q3 MMBT3904, Q4 IRLR8256, Q5 DMN6140L, Q6 MMBT3904, SW1 SW_RST, SW2 SW_BOOT, SW3 On/Off, SW4 Mode, SW5 Up, SW6 Down, U1 AP66200, U2 CP2102N-Axx-xQFN28, U3 USBLC6-2SC6, U4 ESP32-WROOM-32E

Commit message: Board resize in progress
Co-Authored-By: Claude Sonnet 5 <noreply@anthropic.com>
Parts:
- added ?: , , F.Cu at (149.0, 84.0)
- added ?: , , F.Cu at (154.0, 84.0)
- added ?: , , F.Cu at (144.0, 84.0)
- added REF**: Slewform_Logo_20mm, Slewform:Slewform_Logo_20mm, B.Cu at (149.0, 95.0)
- F1: value T3A/63V -> T3A5/63V; footprint Fuse:Fuse_1812_4532Metric -> Fuse:Fuse_1206_3216Metric_Pad1.42x1.75mm_HandSolder
- moved TP2 71.4 mm to (165.1, 103.2)
- moved TP7 68.5 mm to (129.5, 108.3)
- moved TP6 65.9 mm to (132.1, 108.3)
- moved TP1 65.2 mm to (165.1, 108.3)
- moved TP5 63.4 mm to (134.6, 108.3)
- moved TP4 61.2 mm to (137.2, 108.3)
- moved TP3 58.0 mm to (139.7, 108.3)
- moved C10 48.1 mm to (172.1, 85.3)
- moved C11 48.1 mm to (167.8, 95.3)
- moved C6 48.1 mm to (172.6, 91.6)
- moved C8 48.1 mm to (172.6, 95.3)
- moved FB1 48.1 mm to (170.2, 94.7)
- moved L1 48.1 mm to (178.4, 93.7)
- moved C5 47.0 mm to (188.5, 96.0), turned to 0 degrees
- moved R5 46.8 mm to (183.8, 82.3)
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Connections:
- U4 pad 27: unconnected-(U4-IO16-Pad27) -> FAN_PWM
- U4 pad 30: FAN_PWM -> unconnected-(U4-IO18-Pad30)
Routing:
- net 24V_PROT: track 0.00 -> 117.2 mm, vias 0 -> 2
- net 3V3_MCU: track 121.8 -> 55.5 mm, vias 9 -> 14
- net /Power/3V3_BUCK: track 0.00 -> 27.4 mm
- net GND: track 45.6 -> 69.8 mm, vias 25 -> 55
- net Net-(Q2-C): track 36.1 -> 58.1 mm, vias 0 -> 2
- net /MCU/ESP_TXD0: track 26.2 -> 44.0 mm, vias 2 -> 5
- net /MCU/ESP_RXD0: track 26.3 -> 38.6 mm, vias 2 -> 5
- net /Power/VCC_AP66200: track 0.00 -> 11.2 mm, vias 0 -> 3
- net /Power/JACK_24V_RAW: track 0.00 -> 8.26 mm
- net Net-(Q3-C): track 52.6 -> 60.2 mm, vias 2 -> 3
- net Net-(C3-Pad1): track 0.00 -> 7.13 mm
- net Net-(U1-FB): track 0.00 -> 6.73 mm
- net /Power/EN_BUCK: track 0.00 -> 5.16 mm
- net Net-(U1-PG): track 0.00 -> 3.26 mm
- net /MCU/USB_VBUS: track 35.9 -> 38.9 mm
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- added copper zone on In2.Cu, net 3V3_MCU
- added copper zone on In2.Cu, net GND
Other:
- board size 98 x 58 mm -> 95 x 52 mm
