File: hardware/Filament_Dryer_Monitor.kicad_pcb (KiCad board)
At the start: 4 copper layers, 95 x 52 mm, 95 parts, among them J1 DC Connector, J2 USB_C_Receptacle_USB2.0_16P, J3 Sensor, J4 Display, J5 Heater Connector, J6 Fan Connector, J7 NTC Connector, Q1 DMP6180SK3-13, Q2 MMBT3904, Q3 MMBT3904, Q4 IRLR8256, Q5 DMN6140L, Q6 MMBT3904, SW1 SW_RST, SW2 SW_BOOT, SW3 On/Off, SW4 Mode, SW5 Up, SW6 Down, U1 AP66200, U2 CP2102N-Axx-xQFN28, U3 USBLC6-2SC6, U4 ESP32-WROOM-32E

Commit message: Board resize in progress
Parts:
- removed the REF** at (149.0, 95.0)
- Q4: value IRLR8256 -> NTD5865NLT4G
Routing:
- net FAN_PWM: track 52.8 -> 48.6 mm

Commit message: Board resize in progress
Parts:
- U1: footprint Package_DFN_QFN:QFN-16-1EP_4x4mm_P0.65mm_EP2.5x2.5mm -> FilamentDryer:AP66200_U-QFN4040-16_EP2.6x2.6mm_P0.65mm
- U2: footprint Package_DFN_QFN:QFN-28-1EP_5x5mm_P0.5mm_EP3.35x3.35mm -> FilamentDryer:CP2102N_GQFN28_5x5mm_P0.5mm_EP3.35x3.35mm
Routing:
- net GND: track 69.8 -> 69.5 mm, vias 55 -> 50
