File: hardware/Filament_Dryer_Monitor.kicad_pcb (KiCad board)
At the start: 4 copper layers, 95 x 52 mm, 94 parts, among them J1 DC Connector, J2 USB_C_Receptacle_USB2.0_16P, J3 Sensor, J4 Display, J5 Heater Connector, J6 Fan Connector, J7 NTC Connector, Q1 DMP6180SK3-13, Q2 MMBT3904, Q3 MMBT3904, Q4 NTD5865NLT4G, Q5 DMN6140L, Q6 MMBT3904, SW1 SW_RST, SW2 SW_BOOT, SW3 On/Off, SW4 Mode, SW5 Up, SW6 Down, U1 AP66200, U2 CP2102N-Axx-xQFN28, U3 USBLC6-2SC6, U4 ESP32-WROOM-32E

Commit message: Add MPN/LCSC/Manufacturer fields to components; layout WIP
Co-Authored-By: Claude Sonnet 5 <noreply@anthropic.com>
Claude-Session: https://claude.ai/code/session_01TtYFysfg3KHuTv6C83JsmH
Connections:
- U4 pad 13: unconnected-(U4-IO14-Pad13) -> BTN_UP
- U4 pad 14: BTN_UP -> unconnected-(U4-IO12-Pad14)
Routing:
- net BTN_UP: track 67.7 -> 69.0 mm

Commit message: Add MPN/LCSC/Manufacturer fields to components; layout WIP
Co-Authored-By: Claude Sonnet 5 <noreply@anthropic.com>
Claude-Session: https://claude.ai/code/session_019K6fhgSgEV4SPy8guMLbu9
Parts:
- C1: value ~ -> 100n
- C11, C6, C8: value 22u 25V X5R -> 22u
- C5: value 100uF/50V -> 100u
- C7: value 10µF/63V X7R -> 10u
- C9: value 100nF / 50V -> 100n
- F1: value T3A5/63V -> T3A/63V
- Q5: value DMN6140L -> CJ2310
- R2: value ~ -> 7k87
- U2: value CP2102N-Axx-xQFN28 -> CP2102N-A02-GQFN28
- U4: value ESP32-WROOM-32E -> ESP32-WROOM-32E-N4
