File: hardware/Filament_Dryer_Monitor.kicad_pcb (KiCad board)
At the start: 4 copper layers, 95 x 52 mm, 95 parts, among them J1 DC Connector, J2 USB_C_Receptacle_USB2.0_16P, J3 Sensor, J4 Display, J5 Heater Connector, J6 Fan Connector, J7 NTC Connector, Q1 DMP6180SK3-13, Q2 MMBT3904, Q3 MMBT3904, Q4 NTD5865NLT4G, Q5 CJ2310, Q6 MMBT3904, U1 AP66200, U2 CP2102N-A02-GQFN28R, U3 USBLC6-2SC6, U4 ESP32-WROOM-32E-N4

Commit message: Optimize heater MOSFET and NTC input
Co-Authored-By: Claude Sonnet 5 <noreply@anthropic.com>
Parts:
- Q4: value NTD5865NLT4G -> IRLR3636TRPBF
- R28: value 100k -> 47k
Changed lines of the file:
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@@
 			)
 		)
-		(property "Value" "100k"
+		(property "Value" "47k"
 			(at 0 -1.43 270)
 			(layer "B.Fab")
@@
 			)
 		)
-		(property "MPN" "0603WAF1003T5E"
+		(property "MPN" "0603WAF4702T5E"
 			(at 0 0 90)
 			(unlocked yes)
@@
 			)
 		)
-		(property "LCSC" "C25803"
+		(property "LCSC" "C25819"
 			(at 0 0 90)
 			(unlocked yes)
@@
 			)
 		)
-		(property "Value" "NTD5865NLT4G"
+		(property "Value" "IRLR3636TRPBF"
 			(at 0 -4.5 180)
 			(layer "B.Fab")
@@
 			)
 		)
-		(property "Datasheet" "kicad-embed://NTD5865NLT4G.pdf"
+		(property "Datasheet" "kicad-embed://IRLR3636TRPBF.pdf"
 			(at 0 0 180)
 			(layer "B.Fab")
@@
 			)
 		)
-		(property "MPN" "NTD5865NLT4G"
+		(property "MPN" "IRLR3636TRPBF"
 			(at 0 0 0)
 			(unlocked yes)
@@
 			)
 		)
-		(property "LCSC" "C145546"
+		(property "LCSC" "C67279"
 			(at 0 0 0)
 			(unlocked yes)

Commit message: Finalize schematic and PCB revision
Co-Authored-By: Claude Sonnet 5 <noreply@anthropic.com>
Parts:
- REF** (x4): value MountingHole_2.5mm -> MountingHole_2.2mm_M2; footprint MountingHole:MountingHole_2.5mm -> MountingHole:MountingHole_2.2mm_M2
- moved Q6 10.7 mm to (104.4, 87.9)
- moved R22 7.21 mm to (113.0, 110.9)
- moved SW4 7.21 mm to (113.0, 107.0)
- moved REF** 6.80 mm to (107.5, 101.0)
- moved R27 6.49 mm to (104.4, 90.7)
- moved R24 6.40 mm to (171.0, 111.2)
- moved SW6 6.40 mm to (171.0, 107.0)
- moved R19 6.00 mm to (113.0, 98.9)
- moved SW3 6.00 mm to (113.0, 95.0)
- moved REF** 5.85 mm to (118.5, 101.0)
- moved REF** 5.85 mm to (165.5, 101.0)
- moved ? 5.52 mm to (142.0, 84.5)
- moved ? 5.52 mm to (147.0, 84.5)
- moved ? 5.52 mm to (137.0, 84.5)
- moved J4 5.50 mm to (138.2, 88.0)
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Routing:
- net 3V3_MCU: track 65.3 -> 52.3 mm
- net BTN_M: track 14.3 -> 5.66 mm
- net BTN_ONOFF: track 23.5 -> 16.5 mm
- net BUZ_DRV: track 15.6 -> 21.7 mm
- net Net-(D6-A): track 8.91 -> 14.7 mm
- net BTN_UP: track 66.0 -> 61.0 mm
- net Net-(J3-Pin_3): track 100.7 -> 95.8 mm
- net Net-(J3-Pin_2): track 107.9 -> 103.1 mm
- net /MCU/ESP_TXD0: track 44.3 -> 40.5 mm, vias 5 -> 3
- net Net-(Q6-B): track 5.18 -> 1.91 mm
- net HEATER_PWM: track 73.2 -> 70.0 mm
- net FAN_PWM: track 48.6 -> 45.7 mm
- net BTN_DOWN: track 65.6 -> 63.2 mm
- net GND: track 70.1 -> 72.0 mm, vias 47 -> 46
- net 24V_PROT: track 118.7 -> 120.4 mm
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Other:
- board size 95 x 52 mm -> 91 x 52 mm
