File: hardware/IO_Power.kicad_sch (KiCad schematic)
At the start: 25 parts

Commit message: Board resize in progress
Parts:
- BZ1: renamed from BUZZER1; Function (none) -> BUZZER1
- C19: renamed from C_ntc1; Function (none) -> C_ntc1
- D4: renamed from D_heat1; Function (none) -> D_heat1
- D5: renamed from D_fan1; Function (none) -> D_fan1
- D6: renamed from D_buz1; Function (none) -> D_buz1
- J5: renamed from J_heat1; Function (none) -> J_heat1
- J6: renamed from J_fan2; Function (none) -> J_fan2
- J7: renamed from J_ntc1; Function (none) -> J_ntc1
- Q4: renamed from Q_heat1; Function (none) -> Q_heat1
- Q5: renamed from Q_fan1; Function (none) -> Q_fan1
- Q6: renamed from Q_buz1; Function (none) -> Q_buz1
- R19: renamed from R_btn1; Function (none) -> R_btn1
- R20: renamed from R_g_heat1; Function (none) -> R_g_heat1
- R21: renamed from R_pd_heat1; Function (none) -> R_pd_heat1
- R22: renamed from R_btn2; Function (none) -> R_btn2
- R23: renamed from R_btn3; Function (none) -> R_btn3
- R24: renamed from R_btn4; Function (none) -> R_btn4
- R25: renamed from R_g_fan1; Function (none) -> R_g_fan1
- R26: renamed from R_pd_fan1; Function (none) -> R_pd_fan1
- R27: renamed from R_buz1; Function (none) -> R_buz1
- R28: renamed from R_ntc1; Function (none) -> R_ntc1
- SW3: renamed from SW_onoff1; Function (none) -> SW_onoff1
- SW4: renamed from SW_m1; Function (none) -> SW_m1
- SW5: renamed from SW_up1; Function (none) -> SW_up1
- SW6: renamed from SW_down1; Function (none) -> SW_down1

Commit message: Board resize in progress
Parts:
- BZ1: LCSC (none) -> C94599; LCSC Part C94599 -> (none)
- Q4: value IRLR8256 -> NTD5865NLT4G; LCSC (none) -> C145546; MPN (none) -> NTD5865NLT4G; Manufacturer (none) -> onsemi
