File: hardware/IO_Power.kicad_sch (KiCad schematic)
At the start: 25 parts, among them J5 Heater Connector, J6 Fan Connector, J7 NTC Connector, Q4 NTD5865NLT4G, Q5 DMN6140L, Q6 MMBT3904, SW3 On/Off, SW4 Mode, SW5 Up, SW6 Down

Commit message: Add MPN/LCSC/Manufacturer fields to components; layout WIP
Co-Authored-By: Claude Sonnet 5 <noreply@anthropic.com>
Claude-Session: https://claude.ai/code/session_01TtYFysfg3KHuTv6C83JsmH
Parts:
- BZ1: Manufacturer 华能 -> Jiangsu Huaneng Elec
- C19: Dielectric (none) -> X7R; LCSC (none) -> C14663; MPN (none) -> CC0603KRX7R9BB104; Manufacturer (none) -> Yageo; Tolerance (none) -> 10%; Voltage (none) -> 50V
- D4, D5: LCSC (none) -> C98663; MPN (none) -> PMEG6020ER,115; Manufacturer (none) -> Nexperia
- D6: LCSC (none) -> C3313013; MPN (none) -> 1N4148W-G3-18; Manufacturer (none) -> Vishay Intertech
- J5: LCSC (none) -> C158012; MPN (none) -> B2B-XH-A(LF)(SN); Manufacturer (none) -> JST
- J6: LCSC (none) -> C160352; MPN (none) -> B2B-PH-SM4-TB(LF)(SN); Manufacturer (none) -> JST
- J7: LCSC (none) -> C161690; MPN (none) -> BM02B-GHS-TBT(LF)(SN); Manufacturer (none) -> JST
- Q5: value DMN6140L -> CJ2310; LCSC (none) -> C75882; MPN (none) -> CJ2310; Manufacturer (none) -> Jiangsu Changjing Electronics Technology Co., Ltd.
- Q6: LCSC (none) -> C94514; MPN (none) -> MMBT3904-7-F; Manufacturer (none) -> Diodes Incorporated
- R19, R22, R23, R24: LCSC (none) -> C25804; MPN (none) -> 0603WAF1002T5E; Manufacturer (none) -> UNI-ROYAL(Uniroyal Elec); Power (none) -> 100mW; TCR (none) -> 100ppm/K; Tolerance (none) -> 1%
- R20, R25: LCSC (none) -> C22775; MPN (none) -> 0603WAF1000T5E; Manufacturer (none) -> UNI-ROYAL(Uniroyal Elec); Power (none) -> 100mW; TCR (none) -> 100ppm/K; Tolerance (none) -> 1%
- R21, R26, R28: LCSC (none) -> C25803; MPN (none) -> 0603WAF1003T5E; Manufacturer (none) -> UNI-ROYAL(Uniroyal Elec); Power (none) -> 100mW; TCR (none) -> 100ppm/K; Tolerance (none) -> 1%
- R27: LCSC (none) -> C23179; MPN (none) -> 0603WAF4700T5E; Manufacturer (none) -> UNI-ROYAL(Uniroyal Elec); Power (none) -> 100mW; TCR (none) -> 100ppm/K; Tolerance (none) -> 1%
- SW3, SW4, SW5, SW6: LCSC (none) -> C720477; MPN (none) -> TS-1088-AR02016; Manufacturer (none) -> XUNPU

Commit message: Add MPN/LCSC/Manufacturer fields to components; layout WIP
Co-Authored-By: Claude Sonnet 5 <noreply@anthropic.com>
Claude-Session: https://claude.ai/code/session_019K6fhgSgEV4SPy8guMLbu9
Parts:
- D6: LCSC C3313013 -> C81598; MPN 1N4148W-G3-18 -> 1N4148W; Manufacturer Vishay Intertech -> ST(Semtech)
Changed lines of the file:
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@@
 			)
 		)
-		(property "LCSC" "C3313013"
+		(property "LCSC" "C81598"
 			(at 224.79 132.08 90)
 			(hide yes)
@@
 			)
 		)
-		(property "MPN" "1N4148W-G3-18"
+		(property "MPN" "1N4148W"
 			(at 224.79 132.08 90)
 			(hide yes)
@@
 			)
 		)
-		(property "Manufacturer" "Vishay Intertech"
+		(property "Manufacturer" "ST(Semtech)"
 			(at 224.79 132.08 90)
 			(hide yes)
