File: hardware/IO_Power.kicad_sch (KiCad schematic)
At the start: 25 parts, among them J5 Heater Connector, J6 Fan Connector, J7 NTC Connector, Q4 NTD5865NLT4G, Q5 CJ2310, Q6 MMBT3904, SW3 On/Off, SW4 Mode, SW5 Up, SW6 Down

Commit message: Complete PCB layout: first release-ready hardware revision
Finalize board layout, add J3 sensor connector to BOM/position files,
and fix switch label properties (Value/Function swapped for SW1-6).
Parts:
- SW3: value On/Off -> (none); Function SW_onoff1 -> On/Off
- SW4: value Mode -> (none); Function SW_m1 -> Mode
- SW5: value Up -> (none); Function SW_up1 -> Up
- SW6: value Down -> (none); Function SW_down1 -> Down
Changed lines of the file:
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@@
 			)
 		)
-		(property "Value" "Down"
+		(property "Value" ""
 			(at 143.51 144.7799 90)
 			(show_name no)
@@
 			)
 		)
-		(property "Function" "SW_down1"
+		(property "Function" "Down"
 			(at 142.24 143.51 90)
 			(hide yes)
@@
 			)
 		)
-		(property "Value" "Mode"
+		(property "Value" ""
 			(at 95.25 144.7799 90)
 			(show_name no)
@@
 			)
 		)
-		(property "Function" "SW_m1"
+		(property "Function" "Mode"
 			(at 93.98 143.51 90)
 			(hide yes)
@@
 			)
 		)
-		(property "Value" "Up"
+		(property "Value" ""
 			(at 119.38 144.7799 90)
 			(show_name no)
@@
 			)
 		)
-		(property "Function" "SW_up1"
+		(property "Function" "Up"
 			(at 118.11 143.51 90)
 			(hide yes)
@@
 			)
 		)
-		(property "Value" "On/Off"
+		(property "Value" ""
 			(at 71.12 144.7799 90)
 			(show_name no)
@@
 			)
 		)
-		(property "Function" "SW_onoff1"
+		(property "Function" "On/Off"
 			(at 69.85 143.51 90)
 			(hide yes)

Commit message: Add HEATER_SW net label and tighten via design rules
Rename Power_Heat netclass pattern to match the new HEATER_SW label,
reduce min via annular width/diameter, and update PCB layout
accordingly. Add STL export of the board.
Connections:
- net HEATER_SW: now reaches D4.2 (A), J5.1 (Pin_1), Q4.2 (D)
Changed lines of the file:
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@@
+		)
+	)
+	(label "HEATER_SW"
+		(at 87.63 81.28 0)
+		(effects
+			(font
+				(size 1.27 1.27)
+			)
+			(justify left bottom)
 		)
 	)
