File: hardware/IO_Power.kicad_sch (KiCad schematic)
At the start: 25 parts, among them J5 Heater Connector, J6 Fan Connector, J7 NTC Connector, Q4 NTD5865NLT4G, Q5 CJ2310, Q6 MMBT3904

Commit message: Optimize heater MOSFET and NTC input
Co-Authored-By: Claude Sonnet 5 <noreply@anthropic.com>
Parts:
- Q4: value NTD5865NLT4G -> IRLR3636TRPBF; LCSC C145546 -> C67279; MPN NTD5865NLT4G -> IRLR3636TRPBF
- R28: value 100k -> 47k; LCSC C25803 -> C25819; MPN 0603WAF1003T5E -> 0603WAF4702T5E
Changed lines of the file:
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@@
 			)
 		)
-		(property "Value" "100k"
+		(property "Value" "47k"
 			(at 222.25 74.9299 0)
 			(show_name no)
@@
 			)
 		)
-		(property "MPN" "0603WAF1003T5E"
+		(property "MPN" "0603WAF4702T5E"
 			(at 224.79 73.66 0)
 			(hide yes)
@@
 			)
 		)
-		(property "LCSC" "C25803"
+		(property "LCSC" "C25819"
 			(at 224.79 73.66 0)
 			(hide yes)
@@
 			)
 		)
-		(property "Value" "NTD5865NLT4G"
+		(property "Value" "IRLR3636TRPBF"
 			(at 91.44 88.8999 0)
 			(show_name no)
@@
 			)
 		)
-		(property "Datasheet" "kicad-embed://NTD5865NLT4G.pdf"
+		(property "Datasheet" "kicad-embed://IRLR3636TRPBF.pdf"
 			(at 85.09 87.63 0)
 			(hide yes)
@@
 			)
 		)
-		(property "MPN" "NTD5865NLT4G"
+		(property "MPN" "IRLR3636TRPBF"
 			(at 85.09 87.63 0)
 			(hide yes)
@@
 			)
 		)
-		(property "LCSC" "C145546"
+		(property "LCSC" "C67279"
 			(at 85.09 87.63 0)
 			(hide yes)

Commit message: Finalize schematic and PCB revision
Co-Authored-By: Claude Sonnet 5 <noreply@anthropic.com>
Connections:
- no-connect marks 0 -> 2
Changed lines of the file:
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@@
 		(color 0 0 0 0)
+	)
+	(no_connect
+		(at 240.03 139.7)
+	)
+	(no_connect
+		(at 241.3 139.7)
 	)
 	(wire
