File: hardware/IO_Power.kicad_sch (KiCad schematic)
At the start: 25 parts, among them J5 Heater Connector, J6 Fan Connector, J7 NTC Connector, Q4 IRLR3636TRPBF, Q5 CJ2310, Q6 MMBT3904

Commit message: Update components and footprints for Mouser sourcing
Parts:
- BZ1: value MLT-8530 -> CSS-I4B20-SMT-TR; footprint JLCPCB:BUZ-SMD_4P-L8.5-W8.5-P8.50-BR -> CSSI4B20SMTTR; MPN MLT-8530 -> CSS-I4B20-SMT-TR; Manufacturer Jiangsu Huaneng Elec -> Same Sky
- C19: value 100n -> SMBJ28A; footprint Capacitor_SMD:C_0603_1608Metric -> Diode_SMD:D_SMB; Function C_ntc1 -> TVS1; LCSC C14663 -> C96335; MPN CC0603KRX7R9BB104 -> SMBJ28A; Manufacturer Yageo -> Littelfuse
- D4: value PMEG6020ER -> 1N4148W; footprint Diode_SMD:Nexperia_CFP3_SOD-123W -> Diode_SMD:D_SOD-123; Function D_heat1 -> D_buz1; LCSC C98663 -> C81598; MPN PMEG6020ER,115 -> 1N4148W-7-F; Manufacturer Nexperia -> Diodes Incorporated
- D5: value PMEG6020ER -> T3A/63V; footprint Diode_SMD:Nexperia_CFP3_SOD-123W -> Fuse:Fuse_1206_3216Metric_Pad1.42x1.75mm_HandSolder; Function D_fan1 -> F1; LCSC C98663 -> C354897; MPN PMEG6020ER,115 -> SF-1206S300W-2; Manufacturer Nexperia -> Bourns
- D6: value 1N4148W -> HCB3216KF-601T30; footprint Diode_SMD:D_SOD-123 -> Inductor_SMD:L_1206_3216Metric; Function D_buz1 -> FB1; LCSC C81598 -> C357023; MPN 1N4148W -> BLM31KN601SH1L; Manufacturer ST(Semtech) -> Murata Electronics
- J5: value Heater Connector -> 8u2; footprint Connector_JST:JST_XH_B2B-XH-A_1x02_P2.50mm_Vertical -> FilamentDryer:XAL4040-822MEC_HandSolder; Function J_heat1 -> L1; LCSC C158012 -> (none); MPN B2B-XH-A(LF)(SN) -> XAL4040-822MEC; Manufacturer JST -> Coilcraft
- J6: value Fan Connector -> DMP6180SK3-13; footprint FilamentDryer:JST_PH_B2B-PH-SM4-TB_1x02-1MP_P2.00mm_Vertical -> Package_TO_SOT_SMD:TO-252-2; Function J_fan2 -> Q1; LCSC C160352 -> C93034; MPN B2B-PH-SM4-TB(LF)(SN) -> DMP6180SK3-13; Manufacturer JST -> Diodes Incorporated
- J7: value NTC Connector -> MMBT3904; footprint Connector_JST:JST_GH_BM02B-GHS-TBT_1x02-1MP_P1.25mm_Vertical -> Package_TO_SOT_SMD:SOT-23; Function J_ntc1 -> Q_boot1; LCSC C161690 -> C94514; MPN BM02B-GHS-TBT(LF)(SN) -> MMBT3904-7-F; Manufacturer JST -> Diodes Incorporated
- Q4: value IRLR3636TRPBF -> 100k; footprint Package_TO_SOT_SMD:TO-252-2 -> Resistor_SMD:R_0603_1608Metric; Function Q_heat1 -> Ren_top1; LCSC C67279 -> C25803; MPN IRLR3636TRPBF -> RC0603FR-07100KL; Manufacturer onsemi -> YAGEO; Power (none) -> 100mW; Tolerance (none) -> 1%
- Q5: value CJ2310 -> 100k; footprint Package_TO_SOT_SMD:SOT-23 -> Resistor_SMD:R_0603_1608Metric; Function Q_fan1 -> Rg1; LCSC C75882 -> C25803; MPN CJ2310 -> RC0603FR-07100KL; Manufacturer Jiangsu Changjing Electronics Technology Co., Ltd. -> YAGEO; Power (none) -> 100mW; Tolerance (none) -> 1%
- Q6: value MMBT3904 -> 100k; footprint Package_TO_SOT_SMD:SOT-23 -> Resistor_SMD:R_0603_1608Metric; Function Q_buz1 -> Rfb_top1; LCSC C94514 -> C25803; MPN MMBT3904-7-F -> RC0603FR-07100KL; Manufacturer Diodes Incorporated -> YAGEO; Power (none) -> 100mW; Tolerance (none) -> 1%
- R19: Function R_btn1 -> R_btn4; MPN 0603WAF1002T5E -> RC0603FR-0710KL; Manufacturer UNI-ROYAL(Uniroyal Elec) -> YAGEO
- R20: Function R_g_heat1 -> R_g_fan1; MPN 0603WAF1000T5E -> CR0603-FX-1000ELF; Manufacturer UNI-ROYAL(Uniroyal Elec) -> Bourns
- R21: Function R_pd_heat1 -> R_pd_fan1; MPN 0603WAF1003T5E -> RC0603FR-07100KL; Manufacturer UNI-ROYAL(Uniroyal Elec) -> YAGEO
- R22: value 10k -> 470; Function R_btn2 -> R_buz1; LCSC C25804 -> C23179; MPN 0603WAF1002T5E -> RC0603FR-07470RL; Manufacturer UNI-ROYAL(Uniroyal Elec) -> YAGEO
- R23: value 10k -> 47k; Function R_btn3 -> R_ntc1; LCSC C25804 -> C25819; MPN 0603WAF1002T5E -> CRCW060347K0FKEA; Manufacturer UNI-ROYAL(Uniroyal Elec) -> Vishay
- R24: value 10k -> (none); footprint Resistor_SMD:R_0603_1608Metric -> SWT0110020010SSA; Function R_btn4 -> SW_BOOT; LCSC C25804 -> (none); MPN 0603WAF1002T5E -> SWT0110-020010SSA; Manufacturer UNI-ROYAL(Uniroyal Elec) -> GCT
- R25: value 100 -> (none); footprint Resistor_SMD:R_0603_1608Metric -> SWT0110020010SSA; Function R_g_fan1 -> SW_BOOT; LCSC C22775 -> (none); MPN 0603WAF1000T5E -> SWT0110-020010SSA; Manufacturer UNI-ROYAL(Uniroyal Elec) -> GCT
- R26: value 100k -> (none); footprint Resistor_SMD:R_0603_1608Metric -> SWT0110020010SSA; Function R_pd_fan1 -> SW_BOOT; LCSC C25803 -> (none); MPN 0603WAF1003T5E -> SWT0110-020010SSA; Manufacturer UNI-ROYAL(Uniroyal Elec) -> GCT
- R27: value 470 -> (none); footprint Resistor_SMD:R_0603_1608Metric -> SWT0110020010SSA; Function R_buz1 -> SW_BOOT; LCSC C23179 -> (none); MPN 0603WAF4700T5E -> SWT0110-020010SSA; Manufacturer UNI-ROYAL(Uniroyal Elec) -> GCT
- R28: value 47k -> (none); footprint Resistor_SMD:R_0603_1608Metric -> SWT0110020010SSA; Function R_ntc1 -> SW_BOOT; LCSC C25819 -> (none); MPN 0603WAF4702T5E -> SWT0110-020010SSA; Manufacturer UNI-ROYAL(Uniroyal Elec) -> GCT
- SW3: value (none) -> CP2102N-A02-GQFN28R; footprint JLCPCB:SW-SMD_L3.9-W3.0-P4.45 -> FilamentDryer:CP2102N_GQFN28_5x5mm_P0.5mm_EP3.35x3.35mm; Function On/Off -> U3; LCSC C720477 -> C964632; MPN TS-1088-AR02016 -> CP2102N-A02-GQFN28R; Manufacturer XUNPU -> Silicon Labs
- SW4: value (none) -> 82400102; footprint JLCPCB:SW-SMD_L3.9-W3.0-P4.45 -> Package_TO_SOT_SMD:SOT-23-6; Function Mode -> U4; LCSC C720477 -> C7519; MPN TS-1088-AR02016 -> 82400102; Manufacturer XUNPU -> Würth Elektronik
- SW5: value (none) -> ESP32-WROOM-32E-N4; footprint JLCPCB:SW-SMD_L3.9-W3.0-P4.45 -> RF_Module:ESP32-WROOM-32E; Function Up -> U1; LCSC C720477 -> C701341; MPN TS-1088-AR02016 -> ESP32-WROOM-32E-N4; Manufacturer XUNPU -> Espressif Systems
- SW6: footprint JLCPCB:SW-SMD_L3.9-W3.0-P4.45 -> SWT0110020010SSA; Function Down -> SW_BOOT; LCSC C720477 -> (none); MPN TS-1088-AR02016 -> SWT0110-020010SSA; Manufacturer XUNPU -> Tactile Switches Tactile Switch, SPST-NO, 3.9 x 2.93mm, Top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

Commit message: Repair symbol fields after CSV import
Parts:
- BZ1: footprint CSSI4B20SMTTR -> SamacSys_Parts:CSSI4B20SMTTR; LCSC C94599 -> (none)
- C19: value SMBJ28A -> 100n; footprint Diode_SMD:D_SMB -> Capacitor_SMD:C_0603_1608Metric; Function TVS1 -> C_ntc1; LCSC C96335 -> C14663; MPN SMBJ28A -> CC0603KRX7R9BB104; Manufacturer Littelfuse -> YAGEO
- D4: value 1N4148W -> PMEG6020ER; footprint Diode_SMD:D_SOD-123 -> Diode_SMD:Nexperia_CFP3_SOD-123W; Function D_buz1 -> D_heat1; LCSC C81598 -> (none); MPN 1N4148W-7-F -> PMEG6020ER-QX; Manufacturer Diodes Incorporated -> Nexperia
- D5: value T3A/63V -> PMEG6020ER; footprint Fuse:Fuse_1206_3216Metric_Pad1.42x1.75mm_HandSolder -> Diode_SMD:Nexperia_CFP3_SOD-123W; Function F1 -> D_fan1; LCSC C354897 -> (none); MPN SF-1206S300W-2 -> PMEG6020ER-QX; Manufacturer Bourns -> Nexperia
- D6: value HCB3216KF-601T30 -> 1N4148W; footprint Inductor_SMD:L_1206_3216Metric -> Diode_SMD:D_SOD-123; Function FB1 -> D_buz1; LCSC C357023 -> (none); MPN BLM31KN601SH1L -> 1N4148W-7-F; Manufacturer Murata Electronics -> Diodes Incorporated
- J5: value 8u2 -> Heater Connector; footprint FilamentDryer:XAL4040-822MEC_HandSolder -> Connector_JST:JST_XH_B2B-XH-A_1x02_P2.50mm_Vertical; Function L1 -> J_heat1; MPN XAL4040-822MEC -> Kit HALJIA XH-compatible 2P; Manufacturer Coilcraft -> HALJIA
- J6: value DMP6180SK3-13 -> Fan Connector; footprint Package_TO_SOT_SMD:TO-252-2 -> FilamentDryer:JST_PH_B2B-PH-SM4-TB_1x02-1MP_P2.00mm_Vertical; Function Q1 -> J_fan2; LCSC C93034 -> C160352; MPN DMP6180SK3-13 -> B2B-PH-SM4-TB(LF)(SN); Manufacturer Diodes Incorporated -> JST
- J7: value MMBT3904 -> NTC Connector; footprint Package_TO_SOT_SMD:SOT-23 -> Connector_JST:JST_XH_B2B-XH-A_1x02_P2.50mm_Vertical; Function Q_boot1 -> J_ntc1; LCSC C94514 -> (none); MPN MMBT3904-7-F -> Kit HALJIA XH-compatible 2P; Manufacturer Diodes Incorporated -> HALJIA
- Q4: value 100k -> IRLR3636TRPBF; footprint Resistor_SMD:R_0603_1608Metric -> Package_TO_SOT_SMD:TO-252-2; Function Ren_top1 -> Q_heat1; LCSC C25803 -> C67279; MPN RC0603FR-07100KL -> IRLR3636TRPBF; Manufacturer YAGEO -> Infineon; Power 100mW -> (none); Tolerance 1% -> (none)
- Q5: value 100k -> DMN6140L-13; footprint Resistor_SMD:R_0603_1608Metric -> Package_TO_SOT_SMD:SOT-23; Function Rg1 -> Q_fan1; LCSC C25803 -> (none); MPN RC0603FR-07100KL -> DMN6140L-13; Manufacturer YAGEO -> Diodes Incorporated; Power 100mW -> (none); Tolerance 1% -> (none)
- Q6: value 100k -> MMBT3904; footprint Resistor_SMD:R_0603_1608Metric -> Package_TO_SOT_SMD:SOT-23; Function Rfb_top1 -> Q_buz1; LCSC C25803 -> C94514; MPN RC0603FR-07100KL -> MMBT3904-7-F; Manufacturer YAGEO -> Diodes Incorporated; Power 100mW -> (none); Tolerance 1% -> (none)
- R19: Function R_btn4 -> R_btn1; LCSC C25804 -> (none)
- R20: Function R_g_fan1 -> R_g_heat1; LCSC C22775 -> (none)
- R21: Function R_pd_fan1 -> R_pd_heat1; LCSC C25803 -> (none)
- R22: value 470 -> 10k; Function R_buz1 -> R_btn2; LCSC C23179 -> (none); MPN RC0603FR-07470RL -> RC0603FR-0710KL
- R23: value 47k -> 10k; Function R_ntc1 -> R_btn3; LCSC C25819 -> (none); MPN CRCW060347K0FKEA -> RC0603FR-0710KL; Manufacturer Vishay -> YAGEO
- R24: value (none) -> 10k; footprint SWT0110020010SSA -> Resistor_SMD:R_0603_1608Metric; Function SW_BOOT -> R_btn4; MPN SWT0110-020010SSA -> RC0603FR-0710KL; Manufacturer GCT -> YAGEO
- R25: value (none) -> 100; footprint SWT0110020010SSA -> Resistor_SMD:R_0603_1608Metric; Function SW_BOOT -> R_g_fan1; MPN SWT0110-020010SSA -> CR0603-FX-1000ELF; Manufacturer GCT -> Bourns
- R26: value (none) -> 100k; footprint SWT0110020010SSA -> Resistor_SMD:R_0603_1608Metric; Function SW_BOOT -> R_pd_fan1; MPN SWT0110-020010SSA -> RC0603FR-07100KL; Manufacturer GCT -> YAGEO
- R27: value (none) -> 470; footprint SWT0110020010SSA -> Resistor_SMD:R_0603_1608Metric; Function SW_BOOT -> R_buz1; MPN SWT0110-020010SSA -> RC0603FR-07470RL; Manufacturer GCT -> YAGEO
- R28: value (none) -> 47k; footprint SWT0110020010SSA -> Resistor_SMD:R_0603_1608Metric; Function SW_BOOT -> R_ntc1; MPN SWT0110-020010SSA -> CRCW060347K0FKEA; Manufacturer GCT -> Vishay
- SW3: value CP2102N-A02-GQFN28R -> (none); footprint FilamentDryer:CP2102N_GQFN28_5x5mm_P0.5mm_EP3.35x3.35mm -> SamacSys_Parts:SWT0110020010SSA; Function U3 -> On/Off; LCSC C964632 -> (none); MPN CP2102N-A02-GQFN28R -> SWT0110-020010SSA; Manufacturer Silicon Labs -> GCT
- SW4: value 82400102 -> (none); footprint Package_TO_SOT_SMD:SOT-23-6 -> SamacSys_Parts:SWT0110020010SSA; Function U4 -> Mode; LCSC C7519 -> (none); MPN 82400102 -> SWT0110-020010SSA; Manufacturer Würth Elektronik -> GCT
- SW5: value ESP32-WROOM-32E-N4 -> (none); footprint RF_Module:ESP32-WROOM-32E -> SamacSys_Parts:SWT0110020010SSA; Function U1 -> Up; LCSC C701341 -> (none); MPN ESP32-WROOM-32E-N4 -> SWT0110-020010SSA; Manufacturer Espressif Systems -> GCT
- SW6: footprint SWT0110020010SSA -> SamacSys_Parts:SWT0110020010SSA; Function SW_BOOT -> Down; Manufacturer Tactile Switches Tactile Switch, SPST-NO, 3.9 x 2.93mm, Top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 -> GCT

Commit message: Remomved LCSC field
Parts:
- C19: LCSC C14663 -> (none)
- J6: LCSC C160352 -> (none)
- Q4: LCSC C67279 -> (none)
- Q6: LCSC C94514 -> (none)
