File: hardware/IO_Power.kicad_sch (KiCad schematic)
At the start: 26 parts, among them J5 Heater Connector, J6 Fan Connector, J7 NTC Connector, Q4 IRLR3636TRPBF, Q5 CJ2310, Q6 MMBT3904

Commit message: Sync KiCad component metadata with TME BOM
Parts:
- BZ1: LCSC C94599 -> (none); MPN MLT-8530 -> LD-BZEL-T67-0808; Manufacturer Jiangsu Huaneng Elec -> LOUDITY
- C19: LCSC C14663 -> (none); Manufacturer Yageo -> YAGEO
- D4, D5: LCSC C98663 -> (none); Manufacturer Nexperia -> NEXPERIA
- D6: LCSC C81598 -> (none); MPN 1N4148W -> 1N4148WGW; Manufacturer ST(Semtech) -> DIOTEC SEMICONDUCTOR
- J5: LCSC C158012 -> (none); MPN B2B-XH-A(LF)(SN) -> Kit HALJIA XH-compatible 2P; Manufacturer JST -> HALJIA
- J6: LCSC C160352 -> (none); MPN B2B-PH-SM4-TB(LF)(SN) -> B2B-PH-SM4-TB (LF)(SN)
- J7: LCSC C161690 -> (none); MPN BM02B-GHS-TBT(LF)(SN) -> BM02B-GHS-TBT (LF)(SN)(N)
- Q4: LCSC C67279 -> (none); Manufacturer onsemi -> INFINEON TECHNOLOGIES
- Q5: LCSC C75882 -> (none); MPN CJ2310 -> IRLML2060TRPBF; Manufacturer Jiangsu Changjing Electronics Technology Co., Ltd. -> INFINEON TECHNOLOGIES
- Q6: LCSC C94514 -> (none); MPN MMBT3904-7-F -> MMBT3904; Manufacturer Diodes Incorporated -> DIOTEC SEMICONDUCTOR
- R19, R22, R23, R24: LCSC C25804 -> (none); MPN 0603WAF1002T5E -> RC0603FR-0710KL; Manufacturer UNI-ROYAL(Uniroyal Elec) -> YAGEO; Voltage (none) -> 75V
- R20, R25: LCSC C22775 -> (none); MPN 0603WAF1000T5E -> RC0603FR-07100RL; Manufacturer UNI-ROYAL(Uniroyal Elec) -> YAGEO; Voltage (none) -> 75V
- R21, R26: LCSC C25803 -> (none); MPN 0603WAF1003T5E -> RC0603FR-07100KL; Manufacturer UNI-ROYAL(Uniroyal Elec) -> YAGEO; Voltage (none) -> 75V
- R27: LCSC C23179 -> (none); MPN 0603WAF4700T5E -> RC0603FR-07470RL; Manufacturer UNI-ROYAL(Uniroyal Elec) -> YAGEO; Voltage (none) -> 75V
- R28: LCSC C25819 -> (none); MPN 0603WAF4702T5E -> RC0603FR-0747KL; Manufacturer UNI-ROYAL(Uniroyal Elec) -> YAGEO; Voltage (none) -> 75V
- R37: Function R_pd_fan1 -> R_pd_buz1; LCSC C25803 -> (none); MPN 0603WAF1003T5E -> RC0603FR-07100KL; Manufacturer UNI-ROYAL(Uniroyal Elec) -> YAGEO; Voltage (none) -> 75V
- SW3, SW4, SW5, SW6: LCSC C720477 -> (none); MPN TS-1088-AR02016 -> SWT0110-020010SSA; Manufacturer XUNPU -> GCT

Commit message: Close sourced component footprint audit
Parts:
- BZ1: value MLT-8530 -> LD-BZEL-T67-0808; footprint JLCPCB:BUZ-SMD_4P-L8.5-W8.5-P8.50-BR -> FilamentDryer:BUZ_Loudity_SMT67_8.5x8.5
- SW3, SW4, SW5, SW6: footprint JLCPCB:SW-SMD_L3.9-W3.0-P4.45 -> FilamentDryer:SW_GCT_SWT0110
Changed lines of the file:
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@@
 			)
 		)
-		(property "Footprint" "JLCPCB:SW-SMD_L3.9-W3.0-P4.45"
+		(property "Footprint" "FilamentDryer:SW_GCT_SWT0110"
 			(at 137.16 143.51 0)
 			(hide yes)
@@
 			)
 		)
-		(property "Value" "MLT-8530"
+		(property "Value" "LD-BZEL-T67-0808"
 			(at 247.65 133.3499 0)
 			(show_name no)
@@
 			)
 		)
-		(property "Footprint" "JLCPCB:BUZ-SMD_4P-L8.5-W8.5-P8.50-BR"
+		(property "Footprint" "FilamentDryer:BUZ_Loudity_SMT67_8.5x8.5"
 			(at 242.57 147.32 0)
 			(hide yes)
@@
 			)
 		)
-		(property "Footprint" "JLCPCB:SW-SMD_L3.9-W3.0-P4.45"
+		(property "Footprint" "FilamentDryer:SW_GCT_SWT0110"
 			(at 88.9 143.51 0)
 			(hide yes)
@@
 			)
 		)
-		(property "Footprint" "JLCPCB:SW-SMD_L3.9-W3.0-P4.45"
+		(property "Footprint" "FilamentDryer:SW_GCT_SWT0110"
 			(at 113.03 143.51 0)
 			(hide yes)
@@
 			)
 		)
-		(property "Footprint" "JLCPCB:SW-SMD_L3.9-W3.0-P4.45"
+		(property "Footprint" "FilamentDryer:SW_GCT_SWT0110"
 			(at 64.77 143.51 0)
 			(hide yes)

Commit message: Fix strict symbol and pinout mappings
Parts:
- Q5: value CJ2310 -> IRLML2060TRPBF; symbol Transistor_FET:Q_NMOS_GDS -> Transistor_FET:Q_NMOS_GSD
Connections:
- net GND: now also Q5.2 (S); no longer Q5.3 (S)
- net at D5.2 (A), J6.1 (Pin_1): now also Q5.3 (D); no longer Q5.2 (D)
Changed lines of the file:
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@@
 	)
 	(symbol
-		(lib_id "Transistor_FET:Q_NMOS_GDS")
+		(lib_id "Transistor_FET:Q_NMOS_GSD")
 		(at 157.48 87.63 0)
 		(unit 1)
@@
 			)
 		)
-		(property "Value" "CJ2310"
+		(property "Value" "IRLML2060TRPBF"
 			(at 163.83 88.8999 0)
 			(show_name no)
@@
 			)
 		)
-		(property "Datasheet" ""
+		(property "Datasheet" "https://www.infineon.com/dgdl/Infineon-IRLML2060-DataSheet-v01_01-EN.pdf?fileId=5546d462533600a401535664b7fb25ee"
 			(at 157.48 87.63 0)
 			(hide yes)
