File: hardware/MCU.kicad_sch (KiCad schematic)
At the start: 34 parts, among them J2 USB_C_Receptacle_USB2.0_16P, J3 Sensor, J4 Display, Q2 MMBT3904, Q3 MMBT3904, SW1 SW_RST, SW2 SW_BOOT, U2 CP2102N-Axx-xQFN28, U3 USBLC6-2SC6, U4 ESP32-WROOM-32E

Commit message: Add MPN/LCSC/Manufacturer fields to components; layout WIP
Co-Authored-By: Claude Sonnet 5 <noreply@anthropic.com>
Claude-Session: https://claude.ai/code/session_01TtYFysfg3KHuTv6C83JsmH
Parts:
- C12: Dielectric (none) -> X5R; LCSC (none) -> C19666; MPN (none) -> CL10A475KO8NNNC; Manufacturer (none) -> Samsung; Tolerance (none) -> 10%; Voltage (none) -> 16V
- C13, C14, C18: Dielectric (none) -> X7R; LCSC (none) -> C14663; MPN (none) -> CC0603KRX7R9BB104; Manufacturer (none) -> Yageo; Tolerance (none) -> 10%; Voltage (none) -> 50V
- C15, C17: Dielectric (none) -> X7R; LCSC (none) -> C5199872; MPN (none) -> CL10B105KB8NQNC; Manufacturer (none) -> Samsung; Tolerance (none) -> 10%; Voltage (none) -> 50V
- C16: Dielectric (none) -> X5R; LCSC (none) -> C15850; MPN (none) -> CL21A106KAYNNNE; Manufacturer (none) -> Samsung; Tolerance (none) -> 10%; Voltage (none) -> 25V
- D3: LCSC (none) -> C5569446; MPN (none) -> APT2012LZGCK; Manufacturer (none) -> Kingbright
- J2: LCSC (none) -> C165948; MPN (none) -> TYPE-C-31-M-12; Manufacturer (none) -> Korean Hroparts Elec
- J3: LCSC (none) -> C160354; MPN (none) -> B4B-PH-SM4-TB(LF)(SN); Manufacturer (none) -> JST; now left out of the parts list
- J4, TP4, TP5, TP6, TP7: now left out of the parts list
- Q2, Q3: LCSC (none) -> C94514; MPN (none) -> MMBT3904-7-F; Manufacturer (none) -> Diodes Incorporated
- R10, R11: LCSC (none) -> C23186; MPN (none) -> 0603WAF5101T5E; Manufacturer (none) -> UNI-ROYAL(Uniroyal Elec); Power (none) -> 100mW; TCR (none) -> 100ppm/K; Tolerance (none) -> 1%
- R12, R13, R14, R15: LCSC (none) -> C25804; MPN (none) -> 0603WAF1002T5E; Manufacturer (none) -> UNI-ROYAL(Uniroyal Elec); Power (none) -> 100mW; TCR (none) -> 100ppm/K; Tolerance (none) -> 1%
- R16, R17: LCSC (none) -> C23140; MPN (none) -> 0603WAF330JT5E; Manufacturer (none) -> UNI-ROYAL(Uniroyal Elec); Power (none) -> 100mW; TCR (none) -> 100ppm/K; Tolerance (none) -> 1%
- R18: LCSC (none) -> C23138; MPN (none) -> 0603WAF3300T5E; Manufacturer (none) -> UNI-ROYAL(Uniroyal Elec); Power (none) -> 100mW; TCR (none) -> 100ppm/K; Tolerance (none) -> 1%
- R7: LCSC (none) -> C25961; MPN (none) -> 0603WAF2212T5E; Manufacturer (none) -> UNI-ROYAL(Uniroyal Elec); Power (none) -> 100mW; TCR (none) -> 100ppm/K; Tolerance (none) -> 1%
- R8: LCSC (none) -> C23061; MPN (none) -> 0603WAF4752T5E; Manufacturer (none) -> UNI-ROYAL(Uniroyal Elec); Power (none) -> 100mW; TCR (none) -> 100ppm/K; Tolerance (none) -> 1%
- R9: LCSC (none) -> C21190; MPN (none) -> 0603WAF1001T5E; Manufacturer (none) -> UNI-ROYAL(Uniroyal Elec); Power (none) -> 100mW; TCR (none) -> 100ppm/K; Tolerance (none) -> 1%
- SW1, SW2: LCSC (none) -> C720477; MPN (none) -> TS-1088-AR02016; Manufacturer (none) -> XUNPU
- U2: value CP2102N-Axx-xQFN28 -> CP2102N-A02-GQFN28; LCSC (none) -> C1550553; MPN (none) -> CP2102N-A02-GQFN28; Manufacturer (none) -> Skyworks / Silicon Labs
- U3: LCSC (none) -> C7519; MPN (none) -> USBLC6-2SC6; Manufacturer (none) -> STMicroelectronics
- U4: value ESP32-WROOM-32E -> ESP32-WROOM-32E-N4; LCSC (none) -> C701341; MPN (none) -> ESP32-WROOM-32E-N4; Manufacturer (none) -> Espressif Systems
Connections:
- net BTN_UP: now also U4.13 (IO14); no longer U4.14 (IO12)

Commit message: Add MPN/LCSC/Manufacturer fields to components; layout WIP
Co-Authored-By: Claude Sonnet 5 <noreply@anthropic.com>
Claude-Session: https://claude.ai/code/session_019K6fhgSgEV4SPy8guMLbu9
Parts:
- U2: value CP2102N-A02-GQFN28 -> CP2102N-A02-GQFN28R; LCSC C1550553 -> C964632; MPN CP2102N-A02-GQFN28 -> CP2102N-A02-GQFN28R
Changed lines of the file:
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@@
 			)
 		)
-		(property "Value" "CP2102N-A02-GQFN28"
+		(property "Value" "CP2102N-A02-GQFN28R"
 			(at 75.8033 127 0)
 			(show_name no)
@@
 			)
 		)
-		(property "LCSC" "C1550553"
+		(property "LCSC" "C964632"
 			(at 73.66 91.44 0)
 			(hide yes)
@@
 			)
 		)
-		(property "MPN" "CP2102N-A02-GQFN28"
+		(property "MPN" "CP2102N-A02-GQFN28R"
 			(at 73.66 91.44 0)
 			(hide yes)
