File: hardware/MCU.kicad_sch (KiCad schematic)
At the start: 34 parts, among them J2 USB_C_Receptacle_USB2.0_16P, J3 Sensor, J4 Display, Q2 MMBT3904, Q3 MMBT3904, SW1 SW_RST, SW2 SW_BOOT, U2 CP2102N-A02-GQFN28R, U3 USBLC6-2SC6, U4 ESP32-WROOM-32E-N4

Commit message: Complete PCB layout: first release-ready hardware revision
Finalize board layout, add J3 sensor connector to BOM/position files,
and fix switch label properties (Value/Function swapped for SW1-6).
Parts:
- J3: now in the parts list
- SW1: value SW_RST -> (none); Function SW1 -> SW_RST
- SW2: value SW_BOOT -> (none); Function SW2 -> SW_BOOT
Changed lines of the file:
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@@
 			)
 		)
-		(property "Value" "SW_BOOT"
+		(property "Value" ""
 			(at 217.17 69.8499 90)
 			(show_name no)
@@
 			)
 		)
-		(property "Function" "SW2"
+		(property "Function" "SW_BOOT"
 			(at 215.9 68.58 90)
 			(hide yes)
@@
 		(body_style 1)
 		(exclude_from_sim no)
-		(in_bom no)
+		(in_bom yes)
 		(on_board yes)
-		(in_pos_files no)
+		(in_pos_files yes)
 		(dnp no)
 		(property "Reference" "J3"
@@
 			)
 		)
-		(property "Value" "SW_RST"
+		(property "Value" ""
 			(at 156.21 69.8499 90)
 			(show_name no)
@@
 			)
 		)
-		(property "Function" "SW1"
+		(property "Function" "SW_RST"
 			(at 154.94 68.58 90)
 			(hide yes)
