File: hardware/MCU.kicad_sch (KiCad schematic)
At the start: 34 parts, among them J2 USB_C_Receptacle_USB2.0_16P, J3 Sensor, J4 Display, Q2 MMBT3904, Q3 MMBT3904, U2 CP2102N-A02-GQFN28R, U3 USBLC6-2SC6, U4 ESP32-WROOM-32E-N4

Commit message: Finalize schematic and PCB revision
Co-Authored-By: Claude Sonnet 5 <noreply@anthropic.com>
Connections:
- no-connect marks 0 -> 30
Changed lines of the file:
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@@
 		(color 0 0 0 0)
+	)
+	(no_connect
+		(at 199.39 85.09)
+	)
+	(no_connect
+		(at 199.39 72.39)
+	)
+	(no_connect
+		(at 168.91 67.31)
+	)
+	(no_connect
+		(at 168.91 69.85)
+	)
+	(no_connect
+		(at 86.36 86.36)
+	)
+	(no_connect
+		(at 86.36 116.84)
+	)
+	(no_connect
+		(at 86.36 71.12)
+	)
+	(no_connect
+		(at 199.39 90.17)
+	)
+	(no_connect
+		(at 90.17 179.07)
+	)
+	(no_connect
+		(at 86.36 93.98)
+	)
+	(no_connect
+		(at 90.17 176.53)
+	)
+	(no_connect
+		(at 86.36 119.38)
+	)
+	(no_connect
+		(at 199.39 77.47)
+	)
+	(no_connect
+		(at 86.36 73.66)
+	)
+	(no_connect
+		(at 199.39 102.87)
+	)
+	(no_connect
+		(at 86.36 109.22)
+	)
+	(no_connect
+		(at 86.36 104.14)
+	)
+	(no_connect
+		(at 86.36 114.3)
+	)
+	(no_connect
+		(at 86.36 106.68)
+	)
+	(no_connect
+		(at 199.39 105.41)
+	)
+	(no_connect
+		(at 199.39 80.01)
+	)
+	(no_connect
+		(at 86.36 81.28)
+	)
+	(no_connect
+		(at 86.36 99.06)
+	)
+	(no_connect
+		(at 86.36 96.52)
+	)
+	(no_connect
+		(at 199.39 67.31)
+	)
+	(no_connect
+		(at 86.36 101.6)
+	)
+	(no_connect
+		(at 199.39 74.93)
+	)
+	(no_connect
+		(at 86.36 88.9)
+	)
+	(no_connect
+		(at 199.39 92.71)
+	)
+	(no_connect
+		(at 86.36 78.74)
 	)
 	(wire
