File: hardware/MCU.kicad_sch (KiCad schematic)
At the start: 34 parts, among them J2 USB_C_Receptacle_USB2.0_16P, J3 Sensor, J4 Display, Q2 MMBT3904, Q3 MMBT3904, U2 CP2102N-A02-GQFN28R, U3 USBLC6-2SC6, U4 ESP32-WROOM-32E-N4

Commit message: Assign verified footprints for sourced components
Parts:
- J2: footprint FilamentDryer:USB_C_Receptacle_HRO_TYPE-C-31-M-12 -> FilamentDryer:USB_C_GCT_USB4216-03-A
Changed lines of the file:
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@@
 			)
 		)
-		(property "Footprint" "FilamentDryer:USB_C_Receptacle_HRO_TYPE-C-31-M-12"
+		(property "Footprint" "FilamentDryer:USB_C_GCT_USB4216-03-A"
 			(at 78.74 163.83 0)
 			(hide yes)

Commit message: Close sourced component footprint audit
Parts:
- SW1, SW2: footprint JLCPCB:SW-SMD_L3.9-W3.0-P4.45 -> FilamentDryer:SW_GCT_SWT0110
- U2: value CP2102N-A02-GQFN28R -> CP2102-GM; footprint FilamentDryer:CP2102N_GQFN28_5x5mm_P0.5mm_EP3.35x3.35mm -> FilamentDryer:CP2102_GM_QFN28_5x5_P0.5_EP3.25
Changed lines of the file:
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@@
 			)
 		)
-		(property "Value" "CP2102N-A02-GQFN28R"
+		(property "Value" "CP2102-GM"
 			(at 75.8033 127 0)
 			(show_name no)
@@
 			)
 		)
-		(property "Footprint" "FilamentDryer:CP2102N_GQFN28_5x5mm_P0.5mm_EP3.35x3.35mm"
+		(property "Footprint" "FilamentDryer:CP2102_GM_QFN28_5x5_P0.5_EP3.25"
 			(at 106.68 123.19 0)
 			(hide yes)
@@
 			)
 		)
-		(property "Footprint" "JLCPCB:SW-SMD_L3.9-W3.0-P4.45"
+		(property "Footprint" "FilamentDryer:SW_GCT_SWT0110"
 			(at 210.82 68.58 0)
 			(hide yes)
@@
 			)
 		)
-		(property "Footprint" "JLCPCB:SW-SMD_L3.9-W3.0-P4.45"
+		(property "Footprint" "FilamentDryer:SW_GCT_SWT0110"
 			(at 149.86 68.58 0)
 			(hide yes)

Commit message: Fix strict symbol and pinout mappings
Parts:
- U2: symbol Interface_USB:CP2102N-Axx-xQFN28 -> Filament_Dryer_Custom:CP2102-GM
- U3: value USBLC6-2SC6 -> AKS1201
Changed lines of the file:
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@@
 			)
 		)
-		(property "Value" "USBLC6-2SC6"
+		(property "Value" "AKS1201"
 			(at 104.5211 161.29 0)
 			(show_name no)
@@
 	)
 	(symbol
-		(lib_id "Interface_USB:CP2102N-Axx-xQFN28")
+		(lib_id "Filament_Dryer_Custom:CP2102-GM")
 		(at 73.66 91.44 0)
 		(unit 1)
@@
 			)
 		)
-		(property "Datasheet" "https://www.silabs.com/documents/public/data-sheets/cp2102n-datasheet.pdf"
+		(property "Datasheet" "https://www.silabs.com/documents/public/data-sheets/CP2102-9.pdf"
 			(at 74.93 110.49 0)
 			(hide yes)
